File: hardware/CoilX.brd (EAGLE design)
At the start: 30 x 12.7 mm, 13 parts, among them U1 74AHC1G14DBV, U2 TLP283

Commit message: changed zener diode to 75v
Parts:
- D2: value 24V .5W -> 75V .5W
Changed lines of the file:
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@@
 <attribute name="NAME" x="14.605" y="5.207" size="0.8128" layer="25" rot="R180"/>
 </element>
-<element name="D2" library="smt_diodes" package="SOD123" value="24V .5W" x="17.78" y="8.128" smashed="yes" rot="R270">
+<element name="D2" library="smt_diodes" package="SOD123" value="75V .5W" x="17.78" y="8.128" smashed="yes" rot="R270">
 <attribute name="NAME" x="18.78" y="9.228" size="0.8128" layer="25" rot="R270"/>
 </element>

Commit message: updated zener to 110v
Parts:
- D2: value 75V .5W -> 110V .5W
Changed lines of the file:
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@@
 <?xml version="1.0" encoding="utf-8"?>
 <!DOCTYPE eagle SYSTEM "eagle.dtd">
-<eagle version="6.5.0">
+<eagle version="7.2.0">
 <drawing>
 <settings>
@@
 <pass name="Default">
 <param name="RoutingGrid" value="50mil"/>
+<param name="AutoGrid" value="1"/>
+<param name="Efforts" value="0"/>
+<param name="TopRouterVariant" value="1"/>
 <param name="tpViaShape" value="round"/>
 <param name="PrefDir.1" value="|"/>
@@
 <attribute name="NAME" x="14.605" y="5.207" size="0.8128" layer="25" rot="R180"/>
 </element>
-<element name="D2" library="smt_diodes" package="SOD123" value="75V .5W" x="17.78" y="8.128" smashed="yes" rot="R270">
+<element name="D2" library="smt_diodes" package="SOD123" value="110V .5W" x="17.78" y="8.128" smashed="yes" rot="R270">
 <attribute name="NAME" x="18.78" y="9.228" size="0.8128" layer="25" rot="R270"/>
 </element>
